Commit message: adding dry dock vizualization

File: description/dry_dock.urdf (robot description, URDF)
Before this commit: robot dry_dock, 2 links, 1 joints
Joints:
- joint world_to_dock: origin xyz=0 0 0 rpy=0 0 0 -> xyz=0 0 1.35 rpy=0 0 0

Commit message: getting everything Thor compatable

File: description/dry_dock.urdf (robot description, URDF)
Before this commit: robot dry_dock, 2 links, 1 joints
Links:
- link dry_dock_mesh: geometry visual mesh filename=package://sonar_localization/description/beckholmen_boatles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
